File: RS-485.kicad_sch (KiCad schematic)
At the start: 7 parts, among them J10 RJ45, J11 Conn_01x03, J12 Conn_01x04, J16 Conn_01x04, U2 SP3485CN

Commit message: updated schematics etc
Parts:
- removed C1: 0.1uF, SparkFun-Capacitor:C_0603_1608Metric, symbol SparkFun-Capacitor:C
- removed J12: Conn_01x04, symbol Connector_Generic:Conn_01x04
- removed R1: 220, Resistor_SMD:R_0603_1608Metric, symbol Device:R
- removed U2: SP3485CN, Package_SO:SOIC-8_3.9x4.9mm_P1.27mm, symbol Interface_UART:SP3485CN
- added U5: RS485-TTL, Waveshare-TTL-To-RS485-C-Kicad:Waveshare-RS485-TTL, symbol waveshare-rs485-ttl:waveshare-rs485-ttl
- J10: renamed from J16; value Conn_01x04 -> RJ45_PINS; footprint (none) -> Connector_PinHeader_2.54mm:PinHeader_1x04_P2.54mm_Vertical
- J12: renamed from J11; value Conn_01x03 -> RS485-OUT; footprint (none) -> Connector_Phoenix_MC:PhoenixContact_MC_1,5_3-G-3.81_1x03_P3.81mm_Horizontal
- renumbered J10 to J11
Connections:
- net A: now also J12.3 (Pin_3), U5.1 (A+); no longer J12.2 (Pin_2)
- net B: now also J12.2 (Pin_2), U5.2 (B-); no longer J12.3 (Pin_3)
- net GND: now also U5.3 (PE), U5.4 (GND)
- net GPIO0: now also U5.6 (TXD)
- net GPIO1: now also U5.5 (RXD)
- new net 3.3V: U5.7 (VCC)
Other:
- added sheet sp3485 (sp3485.kicad_sch)
- note removed: "Ref: https://www.sparkfun.com/sparkfun-transceiver-breakout-rs-485.html"
- moved on the sheet: J10, J11, J12

Commit message: routing
Parts:
- renumbered J10 to J11, J11 to J12, J12 to J13
Changed lines of the file:
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@@
 		(dnp no)
 		(fields_autoplaced yes)
-		(property "Reference" "#PWR019"
+		(property "Reference" "#PWR024"
 			(at 76.2 64.77 0)
 			(effects
@@
 			(project "ScrapheapPicoPCB"
 				(path "/0a0126d3-e10a-434c-bfa7-71e9aafa3ff9/95a9c5b6-9fe0-49f9-8813-a8150d9a6bbc"
-					(reference "#PWR019")
+					(reference "#PWR024")
 					(unit 1)
 				)
@@
 		(on_board yes)
 		(dnp no)
-		(property "Reference" "J11"
+		(property "Reference" "J12"
 			(at 138.43 50.8 0)
 			(effects
@@
 			(project "ScrapheapPicoPCB"
 				(path "/0a0126d3-e10a-434c-bfa7-71e9aafa3ff9/95a9c5b6-9fe0-49f9-8813-a8150d9a6bbc"
-					(reference "J11")
+					(reference "J12")
 					(unit 1)
 				)
@@
 		(on_board yes)
 		(dnp no)
-		(property "Reference" "J10"
+		(property "Reference" "J11"
 			(at 101.6 30.4801 0)
 			(effects
@@
 			(project "ScrapheapPicoPCB"
 				(path "/0a0126d3-e10a-434c-bfa7-71e9aafa3ff9/95a9c5b6-9fe0-49f9-8813-a8150d9a6bbc"
-					(reference "J10")
+					(reference "J11")
 					(unit 1)
 				)
@@
 		(dnp no)
 		(fields_autoplaced yes)
-		(property "Reference" "#PWR020"
+		(property "Reference" "#PWR025"
 			(at 77.47 46.99 0)
 			(effects
@@
 			(project "ScrapheapPicoPCB"
 				(path "/0a0126d3-e10a-434c-bfa7-71e9aafa3ff9/95a9c5b6-9fe0-49f9-8813-a8150d9a6bbc"
-					(reference "#PWR020")
+					(reference "#PWR025")
 					(unit 1)
 				)
@@
 		(dnp no)
 		(fields_autoplaced yes)
-		(property "Reference" "#PWR026"
+		(property "Reference" "#PWR028"
 			(at 161.29 34.29 0)
 			(effects
@@
 			(project "ScrapheapPicoPCB"
 				(path "/0a0126d3-e10a-434c-bfa7-71e9aafa3ff9/95a9c5b6-9fe0-49f9-8813-a8150d9a6bbc"
-					(reference "#PWR026")
+					(reference "#PWR028")
 					(unit 1)
 				)
@@
 		(on_board yes)
 		(dnp no)
-		(property "Reference" "J12"
+		(property "Reference" "J13"
 			(at 139.7 66.0401 0)
 			(effects
@@
 			(project "ScrapheapPicoPCB"
 				(path "/0a0126d3-e10a-434c-bfa7-71e9aafa3ff9/95a9c5b6-9fe0-49f9-8813-a8150d9a6bbc"
-					(reference "J12")
+					(reference "J13")
 					(unit 1)
 				)
@@
 		(dnp no)
 		(fields_autoplaced yes)
-		(property "Reference" "#PWR025"
+		(property "Reference" "#PWR027"
 			(at 157.48 67.31 0)
 			(effects
@@
 			(project "ScrapheapPicoPCB"
 				(path "/0a0126d3-e10a-434c-bfa7-71e9aafa3ff9/95a9c5b6-9fe0-49f9-8813-a8150d9a6bbc"
-					(reference "#PWR025")
+					(reference "#PWR027")
 					(unit 1)
 				)
@@
 		(dnp no)
 		(fields_autoplaced yes)
-		(property "Reference" "#PWR022"
+		(property "Reference" "#PWR026"
 			(at 116.84 55.88 0)
 			(effects
@@
 			(project "ScrapheapPicoPCB"
 				(path "/0a0126d3-e10a-434c-bfa7-71e9aafa3ff9/95a9c5b6-9fe0-49f9-8813-a8150d9a6bbc"
-					(reference "#PWR022")
-					(unit 1)
-				)
+					(reference "#PWR026")
+					(unit 1)
+				)
