File: ScrapheapPicoPCB.kicad_pcb (KiCad board)
At the start: 2 copper layers, 68.8 x 107.7 mm, 10 parts, among them J1 1, J2 1, J3 Vin, J4 1, J5 1, J6 1, J7 1, J8 1, J9 1, U1 Pico

Commit message: updated schematics etc
Parts:
- removed J9: 1, TerminalBlock_RND:TerminalBlock_RND_205-00295_1x10_P5.08mm_Horizontal
- added C1: 10uF, SparkFun-Capacitor:C_0603_1608Metric, F.Cu at (64.6, 55.2)
- added C10: 10uF, SparkFun-Capacitor:C_0603_1608Metric, F.Cu at (70.8, 74.7)
- added C11: 10uF, SparkFun-Capacitor:C_0603_1608Metric, F.Cu at (70.8, 77.2)
- added C12: 10uF, SparkFun-Capacitor:C_0603_1608Metric, F.Cu at (70.8, 79.7)
- added C13: 10uF, SparkFun-Capacitor:C_0603_1608Metric, F.Cu at (70.8, 82.2)
- added C14: 10uF, SparkFun-Capacitor:C_0603_1608Metric, F.Cu at (70.8, 84.7)
- added C15: 10uF, SparkFun-Capacitor:C_0603_1608Metric, F.Cu at (106.3, 19.2)
- added C2: 10uF, SparkFun-Capacitor:C_0603_1608Metric, F.Cu at (99.7, 92.3)
- added C3: 0.1uF, SparkFun-Capacitor:C_0603_1608Metric, F.Cu at (98.7, 99.1)
- added C4: 0.1uF, SparkFun-Capacitor:C_0603_1608Metric, F.Cu at (73.4, 106.7)
- added C6: 0.1uF, SparkFun-Capacitor:C_0603_1608Metric, F.Cu at (73.1, 116.7)
- added C7: 0.1uF, SparkFun-Capacitor:C_0603_1608Metric, F.Cu at (73.4, 111.8)
- added C8: 10uF, SparkFun-Capacitor:C_0603_1608Metric, F.Cu at (73.4, 114.3)
- added C9: 10uF, SparkFun-Capacitor:C_0603_1608Metric, F.Cu at (70.8, 72.2)
- added D1: SS14, SparkFun-Semiconductor-Standard:SMA, F.Cu at (104.6, 49.2)
- added J10: RJ45_PINS, Connector_PinHeader_2.54mm:PinHeader_1x04_P2.54mm_Vertical, F.Cu at (76.1, 26.6)
- added J11: RJ45, SparkFun-Connector:RJ45-8, F.Cu at (176.9, 165.7)
- added J12: RS485-OUT, Connector_Phoenix_MC:PhoenixContact_MC_1,5_3-G-3.81_1x03_P3.81mm_Horizontal, F.Cu at (154.0, 159.1)
- added J13: TX/RX_CONN, Connector_PinHeader_1.00mm:PinHeader_1x03_P1.00mm_Vertical, F.Cu at (40.3, 55.3)
- added J14: NFC_CONN_0, Connector_JST:JST_XH_B4B-XH-A_1x04_P2.50mm_Vertical, F.Cu at (209.9, 51.0)
- added J15: NFC_CONN_1, Connector_JST:JST_XH_B4B-XH-A_1x04_P2.50mm_Vertical, F.Cu at (195.5, 51.0)
- added J16: NFC_CONN_2, Connector_JST:JST_XH_B4B-XH-A_1x04_P2.50mm_Vertical, F.Cu at (181.1, 51.0)
- added J17: NFC_CONN_3, Connector_JST:JST_XH_B4B-XH-A_1x04_P2.50mm_Vertical, F.Cu at (166.7, 51.0)
- added J18: NFC_CONN_4, Connector_JST:JST_XH_B4B-XH-A_1x04_P2.50mm_Vertical, F.Cu at (152.3, 51.0)
- added J19: NFC_CONN_5, Connector_JST:JST_XH_B4B-XH-A_1x04_P2.50mm_Vertical, F.Cu at (137.9, 51.0)
- added J22: S_PWR1, Connector_Phoenix_MC:PhoenixContact_MC_1,5_2-G-3.81_1x02_P3.81mm_Horizontal, F.Cu at (119.8, 69.2)
- added J23: S_PWR2, Connector_Phoenix_MC:PhoenixContact_MC_1,5_2-G-3.81_1x02_P3.81mm_Horizontal, F.Cu at (212.9, 148.6)
- added J24: Conn_01x02, Connector_PinHeader_2.54mm:PinHeader_1x02_P2.54mm_Vertical, F.Cu at (135.6, 18.0)
- added J25: Conn_01x02, Connector_PinHeader_2.54mm:PinHeader_1x02_P2.54mm_Vertical, F.Cu at (131.9, 18.0)
- added JP1: SolderJumper_2_Bridged, SparkFun-Jumper:Jumper_2_NC_Trace, F.Cu at (110.6, 51.2)
- added JP2: OUT_DIR, Jumper:SolderJumper-3_P1.3mm_Bridged12_Pad1.0x1.5mm, F.Cu at (193.5, 104.7)
- added JP3: IN_DIR, Jumper:SolderJumper-3_P1.3mm_Bridged12_Pad1.0x1.5mm, F.Cu at (83.1, 67.1)
- added NT1: NetTie_2, NetTie:NetTie-2_SMD_Pad0.5mm, F.Cu at (179.9, 72.0)
- added NT2: NetTie_2, NetTie:NetTie-2_SMD_Pad0.5mm, F.Cu at (180.9, 72.0)
- added NT3: NetTie_2, NetTie:NetTie-2_SMD_Pad0.5mm, F.Cu at (181.9, 72.0)
- added NT4: NetTie_2, NetTie:NetTie-2_SMD_Pad0.5mm, F.Cu at (187.9, 93.1)
- added NT5: NetTie_2, NetTie:NetTie-2_SMD_Pad0.5mm, F.Cu at (156.9, 66.0)
- added NT6: NetTie_2, NetTie:NetTie-2_SMD_Pad0.5mm, F.Cu at (68.7, 20.0)
- added NT7: NetTie_2, NetTie:NetTie-2_SMD_Pad0.5mm, F.Cu at (89.9, 19.0)
- added R1: 100R, Resistor_SMD:R_0201_0603Metric_Pad0.64x0.40mm_HandSolder, F.Cu at (124.9, 85.6)
- added R10: 100R, Resistor_SMD:R_0201_0603Metric_Pad0.64x0.40mm_HandSolder, F.Cu at (195.2, 99.2)
- added R11: 100R, Resistor_SMD:R_0201_0603Metric_Pad0.64x0.40mm_HandSolder, F.Cu at (194.5, 93.8)
- added R12: 100R, Resistor_SMD:R_0201_0603Metric_Pad0.64x0.40mm_HandSolder, F.Cu at (199.6, 89.7)
- added R13: 100R, Resistor_SMD:R_0201_0603Metric_Pad0.64x0.40mm_HandSolder, F.Cu at (201.7, 81.7)
- added R14: 100R, Resistor_SMD:R_0201_0603Metric_Pad0.64x0.40mm_HandSolder, F.Cu at (201.2, 79.7)
- added R15: 100R, Resistor_SMD:R_0201_0603Metric_Pad0.64x0.40mm_HandSolder, F.Cu at (201.2, 78.2)
- added R16: 100R, Resistor_SMD:R_0201_0603Metric_Pad0.64x0.40mm_HandSolder, F.Cu at (201.2, 75.2)
- added R18: 4.7k, Resistor_SMD:R_0201_0603Metric_Pad0.64x0.40mm_HandSolder, F.Cu at (235.9, 37.0)
- added R19: 4.7k, Resistor_SMD:R_0201_0603Metric_Pad0.64x0.40mm_HandSolder, F.Cu at (121.9, 23.8)
- added R2: 100R, Resistor_SMD:R_0201_0603Metric_Pad0.64x0.40mm_HandSolder, F.Cu at (124.9, 88.1)
- added R20: 4.7k, Resistor_SMD:R_0201_0603Metric_Pad0.64x0.40mm_HandSolder, F.Cu at (121.9, 22.0)
- added R21: 4.7k, Resistor_SMD:R_0201_0603Metric_Pad0.64x0.40mm_HandSolder, F.Cu at (121.9, 26.8)
- added R22: 4.7k, Resistor_SMD:R_0201_0603Metric_Pad0.64x0.40mm_HandSolder, F.Cu at (121.9, 18.5)
- added R23: 4.7k, Resistor_SMD:R_0201_0603Metric_Pad0.64x0.40mm_HandSolder, F.Cu at (108.0, 40.8)
- added R24: 4.7k, Resistor_SMD:R_0201_0603Metric_Pad0.64x0.40mm_HandSolder, F.Cu at (110.9, 32.0)
- added R25: 4.7k, Resistor_SMD:R_0201_0603Metric_Pad0.64x0.40mm_HandSolder, F.Cu at (110.9, 33.8)
- added R26: 4.7k, Resistor_SMD:R_0201_0603Metric_Pad0.64x0.40mm_HandSolder, F.Cu at (110.9, 35.5)
- added R27: 4.7k, Resistor_SMD:R_0201_0603Metric_Pad0.64x0.40mm_HandSolder, F.Cu at (110.9, 37.2)
- added R28: 4.7k, Resistor_SMD:R_0201_0603Metric_Pad0.64x0.40mm_HandSolder, F.Cu at (110.9, 39.0)
- added R3: 100R, Resistor_SMD:R_0201_0603Metric_Pad0.64x0.40mm_HandSolder, F.Cu at (124.9, 91.6)
- added R31: 4.7k, Resistor_SMD:R_0201_0603Metric_Pad0.64x0.40mm_HandSolder, F.Cu at (113.7, 33.8)
- added R34: 4.7k, Resistor_SMD:R_0201_0603Metric_Pad0.64x0.40mm_HandSolder, F.Cu at (129.4, 85.6)
- added R35: 4.7k, Resistor_SMD:R_0201_0603Metric_Pad0.64x0.40mm_HandSolder, F.Cu at (129.4, 87.4)
- added R36: 4.7k, Resistor_SMD:R_0201_0603Metric_Pad0.64x0.40mm_HandSolder, F.Cu at (129.4, 89.1)
- added R37: 4.7k, Resistor_SMD:R_0201_0603Metric_Pad0.64x0.40mm_HandSolder, F.Cu at (129.4, 90.9)
- added R38: 4.7k, Resistor_SMD:R_0201_0603Metric_Pad0.64x0.40mm_HandSolder, F.Cu at (129.4, 92.6)
- added R39: 4.7k, Resistor_SMD:R_0201_0603Metric_Pad0.64x0.40mm_HandSolder, F.Cu at (129.4, 94.4)
- added R4: 100R, Resistor_SMD:R_0201_0603Metric_Pad0.64x0.40mm_HandSolder, F.Cu at (124.9, 95.1)
- added R40: 4.7k, Resistor_SMD:R_0201_0603Metric_Pad0.64x0.40mm_HandSolder, F.Cu at (129.4, 96.1)
- added R41: 4.7k, Resistor_SMD:R_0201_0603Metric_Pad0.64x0.40mm_HandSolder, F.Cu at (129.4, 97.9)
- added R5: 100R, Resistor_SMD:R_0201_0603Metric_Pad0.64x0.40mm_HandSolder, F.Cu at (124.9, 98.6)
- added R6: 100R, Resistor_SMD:R_0201_0603Metric_Pad0.64x0.40mm_HandSolder, F.Cu at (124.9, 102.1)
- added R7: 100R, Resistor_SMD:R_0201_0603Metric_Pad0.64x0.40mm_HandSolder, F.Cu at (124.9, 105.6)
- added R8: 100R, Resistor_SMD:R_0201_0603Metric_Pad0.64x0.40mm_HandSolder, F.Cu at (124.9, 109.1)
- added R9: 100R, Resistor_SMD:R_0201_0603Metric_Pad0.64x0.40mm_HandSolder, F.Cu at (201.2, 98.7)
- added U2: R-78B3.3-2.0, Converter_DCDC:Converter_DCDC_RECOM_R-78B-2.0_THT, F.Cu at (133.4, 124.8)
- added U3: SN74LVC245APW, Package_SO:SOIC-20W_7.5x12.8mm_P1.27mm, F.Cu at (138.4, 91.1)
- added U4: 74HCT245, Package_SO:SOIC-20W_7.5x12.8mm_P1.27mm, F.Cu at (197.2, 116.2)
- added U5: RS485-TTL, Waveshare-TTL-To-RS485-C-Kicad:Waveshare-RS485-TTL, F.Cu at (168.9, 145.0)
- added U7: 74HC4051, Package_SO:SOIC-16_3.9x9.9mm_P1.27mm, F.Cu at (174.4, 68.0)
- added U8: 74HC4051, Package_SO:SOIC-16_3.9x9.9mm_P1.27mm, F.Cu at (161.8, 68.0)
- J1: footprint TerminalBlock_RND:TerminalBlock_RND_205-00295_1x10_P5.08mm_Horizontal -> Connector_PinHeader_2.54mm:PinHeader_1x10_P2.54mm_Vertical
- J3: value Vin -> PWR_INPUT; footprint TerminalBlock_RND:TerminalBlock_RND_205-00287_1x02_P5.08mm_Horizontal -> Connector_Phoenix_MC:PhoenixContact_MC_1,5_2-G-3.81_1x02_P3.81mm_Horizontal
- J4: value 1 -> VSYS_PICO; footprint TerminalBlock_RND:TerminalBlock_RND_205-00295_1x10_P5.08mm_Horizontal -> Connector_PinHeader_2.54mm:PinHeader_1x02_P2.54mm_Vertical
- J7: value 1 -> SHIFTED_IN_CONN; footprint Connector_PinHeader_2.54mm:PinHeader_1x10_P2.54mm_Vertical -> Connector_Phoenix_MC:PhoenixContact_MC_1,5_8-G-3.81_1x08_P3.81mm_Horizontal
- J8: value 1 -> SHIFTED_OUT_CONN; footprint TerminalBlock_RND:TerminalBlock_RND_205-00295_1x10_P5.08mm_Horizontal -> Connector_Phoenix_MC:PhoenixContact_MC_1,5_8-G-3.81_1x08_P3.81mm_Horizontal
- U1: footprint Pi_Pico_MKME_Lab:RPi_Pico_SMD_TH -> MCU_RaspberryPi_and_Boards:RPi_Pico_SMD_TH
- moved J4 182.7 mm to (75.3, 49.8), turned to 0 degrees
- moved J3 137.0 mm to (119.8, 124.2), turned to -90 degrees
- moved J7 109.7 mm to (119.8, 79.7), turned to -90 degrees
- moved J1 105.9 mm to (185.4, 131.8), turned to 180 degrees
- moved J5 91.5 mm to (149.9, 131.7)
- moved J6 57.9 mm to (149.9, 103.3)
- moved U1 57.5 mm to (167.8, 107.6)
- moved J2 57.2 mm to (185.4, 103.3)
- moved J8 47.6 mm to (212.9, 138.0)
Connections:
- J1 pad 1: GPIO15 -> GPIO0
- J1 pad 10: GPIO8 -> GPIO7
- J1 pad 2: GPIO14 -> GPIO1
- J1 pad 4: GPIO13 -> GPIO2
- J1 pad 5: GPIO12 -> GPIO3
- J1 pad 6: GPIO11 -> GPIO4
- J1 pad 7: GPIO10 -> GPIO5
- J1 pad 9: GPIO9 -> GPIO6
- J3 pad 2: VSYS -> 5V
- J4 pad 1: GPIO7 -> GND
- J4 pad 2: GPIO6 -> VSYS
- J5 pad 1: GPIO0 -> VBUS
- J5 pad 10: GPIO7 -> GPIO26_ADC0
- J5 pad 2: GPIO1 -> VSYS
- J5 pad 4: GPIO2 -> 3V3_EN
- J5 pad 5: GPIO3 -> 3v3_OUT
- J5 pad 6: GPIO4 -> ADC_VREF
- J5 pad 7: GPIO5 -> GPIO28_ADC2
- J5 pad 8: GND -> AGND
- J5 pad 9: GPIO6 -> GPIO27_ADC1
- J7 pad 1: VBUS -> Net-(J7-Pin_1)
- J7 pad 2: VSYS -> Net-(J7-Pin_2)
- J7 pad 3: GND -> Net-(J7-Pin_3)
- J7 pad 4: 3V3_EN -> Net-(J7-Pin_4)
- J7 pad 5: 3v3 -> Net-(J7-Pin_5)
- J7 pad 6: ADC_VREF -> Net-(J7-Pin_6)
- J7 pad 7: GPIO28_ADC2 -> Net-(J7-Pin_7)
- J7 pad 8: AGND -> Net-(J7-Pin_8)
- J8 pad 1: RUN -> Net-(J8-Pin_1)
- J8 pad 2: GPIO22 -> Net-(J8-Pin_2)
- J8 pad 3: GND -> Net-(J8-Pin_3)
- J8 pad 4: GPIO21 -> Net-(J8-Pin_4)
- J8 pad 5: GPIO20 -> Net-(J8-Pin_5)
- J8 pad 6: GPIO19 -> Net-(J8-Pin_6)
- J8 pad 7: GPIO18 -> Net-(J8-Pin_7)
- J8 pad 8: GND -> Net-(J8-Pin_8)
- U1 pad 36: 3v3 -> 3v3_OUT
- U1 pad 41: Net-(U1-Pad41) -> unconnected-(U1-SWCLK-Pad41)_1
- U1 pad 42: GND -> unconnected-(U1-GND-Pad42)
- U1 pad 43: Net-(U1-Pad43) -> unconnected-(U1-SWDIO-Pad43)_1
Routing:
- net GND: track 315.5 -> 0.00 mm
- net VSYS: track 149.7 -> 0.00 mm
- net GPIO15: track 65.8 -> 0.00 mm
- net GPIO14: track 62.8 -> 0.00 mm
- net GPIO13: track 55.5 -> 0.00 mm
- net GPIO12: track 52.8 -> 0.00 mm
- net GPIO16: track 64.3 -> 11.6 mm
- net GPIO17: track 61.5 -> 10.3 mm
- net GPIO11: track 50.3 -> 0.03 mm
- net GPIO18: track 55.7 -> 7.87 mm
- net GPIO10: track 47.7 -> 0.00 mm
- net GPIO19: track 53.1 -> 7.34 mm
- net NFC_TX_5: track 0.00 -> 43.9 mm
- net GPIO20: track 50.6 -> 6.88 mm
- net GPIO9: track 42.7 -> 0.00 mm
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Other:
- board size 68.8 x 107.7 mm -> 101.9 x 120.2 mm
- board text removed: "- +"
- board text removed: "PI PICO BREAKOUT V2"
- board text removed: "PI PICO BREAKOUT V2.0"
- board text removed: "Vin"
- board text removed: "WWW.MKME.ORG"

Commit message: routing
Parts:
- removed C15: 10uF, SparkFun-Capacitor:C_0603_1608Metric
- removed the J22 at (119.8, 69.2)
- removed NT3, NT4, NT5, NT6, NT7: NetTie_2, NetTie:NetTie-2_SMD_Pad0.5mm
- removed R37, R38, R39, R40, R41: 4.7k, Resistor_SMD:R_0201_0603Metric_Pad0.64x0.40mm_HandSolder
- added C5: 0.1uF, SparkFun-Capacitor:C_0603_1608Metric, F.Cu at (1.50, 32.3)
- added H1: MountingHole, MountingHole:MountingHole_3.2mm_M3, F.Cu at (121.9, 53.0)
- added H2: MountingHole, MountingHole:MountingHole_3.2mm_M3, F.Cu at (214.3, 52.5)
- added H3: MountingHole, MountingHole:MountingHole_3.2mm_M3, F.Cu at (121.4, 145.5)
- added H4: MountingHole, MountingHole:MountingHole_3.2mm_M3, F.Cu at (214.4, 145.5)
- added J14: Conn_01x01, Connector_PinHeader_2.54mm:PinHeader_1x01_P2.54mm_Vertical, F.Cu at (232.4, 66.2)
- added J15: Conn_01x01, Connector_PinHeader_2.54mm:PinHeader_1x01_P2.54mm_Vertical, F.Cu at (232.4, 70.8)
- added J16: Conn_01x01, Connector_PinHeader_2.54mm:PinHeader_1x01_P2.54mm_Vertical, F.Cu at (232.4, 75.4)
- added J26: Conn_01x01, Connector_PinHeader_2.54mm:PinHeader_1x01_P2.54mm_Vertical, F.Cu at (237.0, 75.4)
- added J9: SHIFTED_OUT_CONN, Connector_Phoenix_MC:PhoenixContact_MC_1,5_8-G-3.81_1x08_P3.81mm_Horizontal, F.Cu at (210.9, 98.3)
- added R17: 100R, Resistor_SMD:R_0201_0603Metric_Pad0.64x0.40mm_HandSolder, F.Cu at (0.91, 12.6)
- added R29: 4.7k, Resistor_SMD:R_0201_0603Metric_Pad0.64x0.40mm_HandSolder, F.Cu at (15.4, 16.3)
- added R30: 4.7k, Resistor_SMD:R_0201_0603Metric_Pad0.64x0.40mm_HandSolder, F.Cu at (15.4, 18.1)
- added R32: 4.7k, Resistor_SMD:R_0201_0603Metric_Pad0.64x0.40mm_HandSolder, F.Cu at (15.4, 19.8)
- added R33: 4.7k, Resistor_SMD:R_0201_0603Metric_Pad0.64x0.40mm_HandSolder, F.Cu at (15.4, 21.6)
- C7: value 0.1uF -> 10uF
- J10: value RJ45_PINS -> S_PWR2; footprint Connector_PinHeader_2.54mm:PinHeader_1x04_P2.54mm_Vertical -> Connector_Phoenix_MC:PhoenixContact_MC_1,5_2-G-3.81_1x02_P3.81mm_Horizontal
- J11: value RJ45 -> RJ45_PINS; footprint SparkFun-Connector:RJ45-8 -> Connector_PinHeader_2.54mm:PinHeader_1x04_P2.54mm_Vertical
- J12: value RS485-OUT -> RJ45; footprint Connector_Phoenix_MC:PhoenixContact_MC_1,5_3-G-3.81_1x03_P3.81mm_Horizontal -> SparkFun-Connector:RJ45-8
- J13: value TX/RX_CONN -> RS485-OUT; footprint Connector_PinHeader_1.00mm:PinHeader_1x03_P1.00mm_Vertical -> Connector_Phoenix_MC:PhoenixContact_MC_1,5_3-G-3.81_1x03_P3.81mm_Horizontal
- J23: value S_PWR2 -> Conn_01x01; footprint Connector_Phoenix_MC:PhoenixContact_MC_1,5_2-G-3.81_1x02_P3.81mm_Horizontal -> Connector_PinHeader_2.54mm:PinHeader_1x01_P2.54mm_Vertical
- J24, J25: value Conn_01x02 -> Conn_01x01; footprint Connector_PinHeader_2.54mm:PinHeader_1x02_P2.54mm_Vertical -> Connector_PinHeader_2.54mm:PinHeader_1x01_P2.54mm_Vertical
- J8: value SHIFTED_OUT_CONN -> S_PWR1; footprint Connector_Phoenix_MC:PhoenixContact_MC_1,5_8-G-3.81_1x08_P3.81mm_Horizontal -> Connector_Phoenix_MC:PhoenixContact_MC_1,5_2-G-3.81_1x02_P3.81mm_Horizontal
- JP2: value OUT_DIR -> IN_DIR
- JP3: value IN_DIR -> OUT_DIR
- R1, R2, R3, R4, R5, R6, R7, R8: value 100R -> 4.7k
- R18, R19, R20, R21, R22, R23, R24: value 4.7k -> 100R
- moved J13 183.9 mm to (210.9, 124.0), turned to 90 degrees
- moved NT2 172.3 mm to (15.2, 24.7), turned to 0 degrees
- moved NT1 171.7 mm to (15.2, 23.2), turned to 0 degrees
- moved J10 158.0 mm to (210.9, 108.8), turned to 90 degrees
- moved J25 117.6 mm to (237.0, 70.8), turned to 0 degrees
- moved J24 112.2 mm to (237.0, 66.2), turned to 0 degrees
- moved J8 111.0 mm to (125.8, 69.2), turned to -90 degrees
- moved R23 98.0 mm to (203.9, 61.5)
- moved R19 92.0 mm to (203.4, 66.5)
- moved R24 87.1 mm to (191.5, 65.0)
- moved J23 71.3 mm to (232.4, 80.0), turned to 0 degrees
- moved R25 67.8 mm to (174.0, 58.5)
- moved J12 62.3 mm to (211.9, 136.0), turned to 90 degrees
- moved R20 59.9 mm to (169.4, 58.5)
- moved U2 54.0 mm to (133.4, 70.8)
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- renumbered J14 to J17, J15 to J18, J16 to J19, J17 to J20, J18 to J21, J19 to J22, U7 to U6, U8 to U7
Connections:
- J10 pad 1: 1 -> GND
- J10 pad 2: 2 -> 5V
- J11 pad 4: GND -> 4
- J12 pad 1: GND -> 1
- J12 pad 2: B -> 2
- J12 pad 3: A -> 3
- J13 pad 2: MUX_TX -> B
- J13 pad 3: MUX_RX -> A
- J23 pad 1: GND -> NFC_TX_6
- J24 pad 1: NFC_TX_6 -> NFC_RX_6
- J8 pad 1: Net-(J8-Pin_1) -> GND
- J8 pad 2: Net-(J8-Pin_2) -> 5V
- JP2 pad 1: 5V -> GND
- JP2 pad 3: GND -> 3.3V
- JP3 pad 1: GND -> 5V
- JP3 pad 3: 3.3V -> GND
- NT1 pad 1: GPIO13 -> 3.3V
- NT1 pad 2: S0 -> 3.3V
- NT2 pad 1: GPIO14 -> GND
- NT2 pad 2: S1 -> GND
- R1 pad 1: Net-(J7-Pin_1) -> IN0
- R1 pad 2: IN0 -> 5V
- R10 pad 1: OUT1 -> Net-(J7-Pin_2)
- R10 pad 2: Net-(J8-Pin_2) -> IN1
- R11 pad 1: OUT2 -> Net-(J7-Pin_3)
- R11 pad 2: Net-(J8-Pin_3) -> IN2
- R12 pad 1: OUT3 -> Net-(J7-Pin_4)
- R12 pad 2: Net-(J8-Pin_4) -> IN3
- R13 pad 1: OUT4 -> Net-(J7-Pin_5)
- R13 pad 2: Net-(J8-Pin_5) -> IN4
- R14 pad 1: OUT5 -> Net-(J7-Pin_6)
- R14 pad 2: Net-(J8-Pin_6) -> IN5
- R15 pad 1: OUT6 -> Net-(J7-Pin_7)
- R15 pad 2: Net-(J8-Pin_7) -> IN6
- R16 pad 1: OUT7 -> Net-(J7-Pin_8)
- R16 pad 2: Net-(J8-Pin_8) -> IN7
- R18 pad 1: 3.3V -> OUT1
- R18 pad 2: NFC_TX_0 -> Net-(J9-Pin_2)
- R19 pad 1: 3.3V -> OUT2
- R19 pad 2: NFC_TX_1 -> Net-(J9-Pin_3)
- R2 pad 1: Net-(J7-Pin_2) -> IN1
- R2 pad 2: IN1 -> 5V
- R20 pad 1: 3.3V -> OUT3
- R20 pad 2: NFC_TX_2 -> Net-(J9-Pin_4)
- R21 pad 1: 3.3V -> OUT4
- R21 pad 2: NFC_TX_3 -> Net-(J9-Pin_5)
- R22 pad 1: 3.3V -> OUT5
- R22 pad 2: NFC_TX_4 -> Net-(J9-Pin_6)
- R23 pad 1: 3.3V -> OUT6
- R23 pad 2: NFC_RX_0 -> Net-(J9-Pin_7)
- R24 pad 1: 3.3V -> OUT7
- R24 pad 2: NFC_RX_1 -> Net-(J9-Pin_8)
- R25 pad 2: NFC_RX_2 -> NFC_TX_0
- R26 pad 2: NFC_RX_3 -> NFC_TX_1
- R27 pad 2: NFC_RX_4 -> NFC_TX_2
- R28 pad 2: NFC_TX_5 -> NFC_TX_3
- R3 pad 1: Net-(J7-Pin_3) -> IN2
- R3 pad 2: IN2 -> 5V
- R31 pad 2: NFC_RX_5 -> NFC_RX_1
- R34 pad 1: IN0 -> 3.3V
- R34 pad 2: 5V -> NFC_RX_4
- R35 pad 1: IN1 -> 3.3V
- R35 pad 2: 5V -> NFC_TX_5
- R36 pad 1: IN2 -> 3.3V
- R36 pad 2: 5V -> NFC_RX_5
- R4 pad 1: Net-(J7-Pin_4) -> IN3
- R4 pad 2: IN3 -> 5V
- R5 pad 1: Net-(J7-Pin_5) -> IN4
- R5 pad 2: IN4 -> 5V
- R6 pad 1: Net-(J7-Pin_6) -> IN5
- R6 pad 2: IN5 -> 5V
- R7 pad 1: Net-(J7-Pin_7) -> IN6
- R7 pad 2: IN6 -> 5V
- R8 pad 1: Net-(J7-Pin_8) -> IN7
- R8 pad 2: IN7 -> 5V
- R9 pad 1: OUT0 -> Net-(J7-Pin_1)
- R9 pad 2: Net-(J8-Pin_1) -> IN0
- U3 pad 1: Net-(JP3-C) -> Net-(JP2-C)
- U4 pad 1: Net-(JP2-C) -> Net-(JP3-C)
- U6 pad 10: S1 -> GPIO14
- U6 pad 11: S0 -> GPIO13
- U6 pad 12: NFC_TX_0 -> NFC_TX_3
- U6 pad 13: NFC_TX_1 -> NFC_TX_0
- U6 pad 14: NFC_TX_2 -> NFC_TX_1
- U6 pad 15: NFC_TX_3 -> NFC_TX_2
- U6 pad 2: NFC_TX_5 -> NFC_TX_6
- U6 pad 3: MUX_TX -> GPIO11
- U6 pad 4: NFC_TX_6 -> NFC_TX_7
- U6 pad 5: NFC_TX_7 -> NFC_TX_5
- U6 pad 9: S2 -> GPIO15
- U7 pad 10: S1 -> GPIO14
- U7 pad 11: S0 -> GPIO13
- U7 pad 12: NFC_RX_0 -> NFC_RX_3
- U7 pad 13: NFC_RX_1 -> NFC_RX_0
- U7 pad 14: NFC_RX_2 -> NFC_RX_1
- U7 pad 15: NFC_RX_3 -> NFC_RX_2
- U7 pad 2: NFC_RX_5 -> NFC_RX_6
- U7 pad 3: MUX_RX -> GPIO12
- U7 pad 4: NFC_RX_6 -> NFC_RX_7
- U7 pad 5: NFC_RX_7 -> NFC_RX_5
- U7 pad 9: S2 -> GPIO15
Routing:
- net GPIO11: track 0.03 -> 53.8 mm, vias 0 -> 2
- net GPIO13: track 0.00 -> 51.1 mm, vias 0 -> 2
- net GPIO12: track 0.00 -> 45.9 mm
- net GPIO14: track 0.00 -> 45.2 mm, vias 0 -> 2
- net NFC_RX_0: track 0.00 -> 45.2 mm
- net NFC_TX_5: track 43.9 -> 9.29 mm, vias 0 -> 1
- net GPIO15: track 0.00 -> 32.1 mm
- net NFC_RX_1: track 13.5 -> 30.2 mm, vias 1 -> 0
- net GPIO26_ADC0: track 15.6 -> 0.00 mm
- net GPIO16: track 11.6 -> 0.00 mm
- net GPIO17: track 10.3 -> 0.00 mm
- net GPIO22: track 10.2 -> 0.00 mm
- net GPIO9: track 0.00 -> 9.97 mm
- net GPIO8: track 0.00 -> 9.97 mm
- net GPIO10: track 0.00 -> 9.97 mm
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Other:
- board size 101.9 x 120.2 mm -> 100 x 100 mm
