File: ScrapheapPicoPCB.kicad_sch (KiCad schematic)
At the start: 17 parts, among them J1 1, J13 Conn_01x03, J17 Conn_01x08, J18 Conn_01x08, J2 1, J3 Vin, J4 1, J5 1, J6 1, J7 1, J8 1, J9 1, U1 Pico, U6 SN74LVC245APW, U7 74HCT245

Commit message: updated schematics etc
Parts:
- removed J1, J4, J8, J9: 1, TerminalBlock_RND:TerminalBlock_RND_205-00295_1x10_P5.08mm_Horizontal, symbol Connector:Screw_Terminal_01x10
- removed J13: Conn_01x03, symbol Connector_Generic:Conn_01x04
- removed J3: Vin, TerminalBlock_RND:TerminalBlock_RND_205-00287_1x02_P5.08mm_Horizontal, symbol Connector:Screw_Terminal_01x02
- added C1, C2: 10uF, SparkFun-Capacitor:C_0603_1608Metric, symbol SparkFun-Capacitor:C
- added D1: SS14, SparkFun-Semiconductor-Standard:SMA, symbol SparkFun-DiscreteSemi:D_Schottky_1A_40V_0.5V
- added J22: S_PWR1, Connector_Phoenix_MC:PhoenixContact_MC_1,5_2-G-3.81_1x02_P3.81mm_Horizontal, symbol Connector_Generic:Conn_01x02
- added J23: S_PWR2, Connector_Phoenix_MC:PhoenixContact_MC_1,5_2-G-3.81_1x02_P3.81mm_Horizontal, symbol Connector_Generic:Conn_01x02
- added J3: PWR_INPUT, Connector_Phoenix_MC:PhoenixContact_MC_1,5_2-G-3.81_1x02_P3.81mm_Horizontal, symbol Connector_Generic:Conn_01x02
- added J4: VSYS_PICO, Connector_PinHeader_2.54mm:PinHeader_1x02_P2.54mm_Vertical, symbol Connector_Generic:Conn_01x02
- added JP1: SolderJumper_2_Bridged, SparkFun-Jumper:Jumper_2_NC_Trace, symbol Jumper:SolderJumper_2_Bridged
- added JP2: OUT_DIR, Jumper:SolderJumper-3_P1.3mm_Bridged12_Pad1.0x1.5mm, symbol Jumper:SolderJumper_3_Bridged12
- added JP3: IN_DIR, Jumper:SolderJumper-3_P1.3mm_Bridged12_Pad1.0x1.5mm, symbol Jumper:SolderJumper_3_Bridged12
- added R1, R10, R11, R12, R13, R14, R15, R16, R2, R3, R4, R5, R6, R7, R8, R9: 100R, Resistor_SMD:R_0201_0603Metric_Pad0.64x0.40mm_HandSolder, symbol Device:R
- added R34, R35, R36, R37, R38, R39, R40, R41: 4.7k, Resistor_SMD:R_0201_0603Metric_Pad0.64x0.40mm_HandSolder, symbol Device:R
- added U2: R-78B3.3-2.0, Converter_DCDC:Converter_DCDC_RECOM_R-78B-2.0_THT, symbol Converter_DCDC:R-78B3.3-2.0
- J7: renamed from J18; value Conn_01x08 -> SHIFTED_IN_CONN; footprint (none) -> Connector_Phoenix_MC:PhoenixContact_MC_1,5_8-G-3.81_1x08_P3.81mm_Horizontal
- J8: renamed from J17; value Conn_01x08 -> SHIFTED_OUT_CONN; footprint (none) -> Connector_Phoenix_MC:PhoenixContact_MC_1,5_8-G-3.81_1x08_P3.81mm_Horizontal
- U1: footprint Pi_Pico_MKME_Lab:RPi_Pico_SMD_TH -> MCU_RaspberryPi_and_Boards:RPi_Pico_SMD_TH
- U3: renamed from U6; footprint Package_SO:TSSOP-20_4.4x6.5mm_P0.65mm -> Package_SO:SOIC-20W_7.5x12.8mm_P1.27mm
- U4: renamed from U7; footprint Package_SO:TSSOP-20_4.4x6.5mm_P0.65mm -> Package_SO:SOIC-20W_7.5x12.8mm_P1.27mm
- renumbered C4 to C3, C5 to C4, J5 to J1, J7 to J5
Connections:
- net GND: now also C1.2, C2.2, J22.1 (Pin_1), J23.1 (Pin_1), J3.1 (Pin_1), J4.1 (Pin_1), JP2.3 (B), JP3.1 (A), U2.2 (GND); no longer U1.42 (GND)
- net GPIO16: now also U3.18 (B1)
- net GPIO17: now also U3.17 (B2)
- net GPIO18: now also U3.16 (B3)
- net GPIO19: now also U3.15 (B4)
- net GPIO2: now also U4.9 (A7)
- net GPIO20: now also U3.14 (B5)
- net GPIO21: now also U3.13 (B6)
- net GPIO22: now also U3.12 (B7)
- net GPIO26_ADC0: now also U3.11 (B8)
- net GPIO3: now also U4.8 (A6)
- net GPIO4: now also U4.7 (A5)
- net GPIO5: now also U4.6 (A4)
- net GPIO6: now also U4.5 (A3)
- net GPIO7: now also U4.4 (A2)
- net GPIO8: now also U4.3 (A1)
- net GPIO9: now also U4.2 (A0)
- net VSYS: now also J4.2 (Pin_2), JP1.1 (A)
- net at J7.1 (Pin_1): now also R1.1; no longer U3.2 (A1)
- net at J7.2 (Pin_2): now also R2.1; no longer U3.3 (A2)
- net at J7.3 (Pin_3): now also R3.1; no longer U3.4 (A3)
- net at J7.4 (Pin_4): now also R4.1; no longer U3.5 (A4)
- net at J7.5 (Pin_5): now also R5.1; no longer U3.6 (A5)
- net at J7.6 (Pin_6): now also R6.1; no longer U3.7 (A6)
- net at J7.7 (Pin_7): now also R7.1; no longer U3.8 (A7)
- net at J7.8 (Pin_8): now also R8.1; no longer U3.9 (A8)
- net at J8.1 (Pin_1): now also R9.2; no longer U4.11 (B7)
- net at J8.2 (Pin_2): now also R10.2; no longer U4.12 (B6)
- net at J8.3 (Pin_3): now also R11.2; no longer U4.13 (B5)
- net at J8.4 (Pin_4): now also R12.2; no longer U4.14 (B4)
- net at J8.5 (Pin_5): now also R13.2; no longer U4.15 (B3)
- net at J8.6 (Pin_6): now also R14.2; no longer U4.16 (B2)
- net at J8.7 (Pin_7): now also R15.2; no longer U4.17 (B1)
- net at J8.8 (Pin_8): now also R16.2; no longer U4.18 (B0)
- net 3.3v renamed 3.3V
- net 3.3V: now also C2.1, JP3.3 (B), U2.3 (OUT); no longer U3.1 (DIR)
- net 3v3 renamed 3v3_OUT
- net 5v renamed 5V
- net 5V: now also C1.1, D1.2 (A), J22.2 (Pin_2), J23.2 (Pin_2), J3.2 (Pin_2), JP2.1 (A), R34.2, R35.2, R36.2, R37.2, R38.2, R39.2, R40.2, R41.2, U2.1 (IN); no longer U4.1 (A->B)
- net SWCLK: no longer names the net of U1.41 (SWCLK)
- net SWDIO: no longer names the net of U1.43 (SWDIO)
- new net: JP3.2 (C), U3.1 (DIR)
- new net: D1.1 (K), JP1.2 (B)
- new net: JP2.2 (C), U4.1 (A->B)
- new net IN0: R1.2, R34.1, U3.2 (A1)
- new net IN1: R2.2, R35.1, U3.3 (A2)
- new net IN2: R3.2, R36.1, U3.4 (A3)
- new net IN3: R37.1, R4.2, U3.5 (A4)
- new net IN4: R38.1, R5.2, U3.6 (A5)
- new net IN5: R39.1, R6.2, U3.7 (A6)
- new net IN6: R40.1, R7.2, U3.8 (A7)
- new net IN7: R41.1, R8.2, U3.9 (A8)
- new net OUT0: R9.1, U4.11 (B7)
- new net OUT1: R10.1, U4.12 (B6)
- new net OUT2: R11.1, U4.13 (B5)
- new net OUT3: R12.1, U4.14 (B4)
- new net OUT4: R13.1, U4.15 (B3)
- new net OUT5: R14.1, U4.16 (B2)
- new net OUT6: R15.1, U4.17 (B1)
- new net OUT7: R16.1, U4.18 (B0)
- no-connect marks 1 -> 3
Other:
- note added: "POWER SUPPLY (VBUS) 5v Power in from USB (VSYS) 5v Power in externally (3V3_OUT) 3.3v Regulated by Pico for powering RP2040 5v Ext Power In 3.3v Regulated Board Power for logic and electronics. Need a power input connector on the board (5v). The Pico can generate its own 3.3v from this, but the input needs to be protected with a shottkey diode to prevent backfeeding the USB as per datasheet PAGE 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"
- note added: "Pico -> 5v TTL For Relays, NeoPixels etc"
- note removed: "POWER SUPPLY -5v Power in from USB -5v Power in externally -3.3v Regulated by Pico for powering RP2040 -3.3v for on board logic and electronics. Need a power input connector on the board (5v). The Pico can generate its own 3.3v from this, but the input needs to be protected with a shottkey diode to prevent backfeeding the USB as per datasheet PAGE 22 (https://pip-assets.raspberrypi.com/categories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"
- note removed: "Pico -> 5v TTL For NeoPixels etc"
- moved on the sheet: C3, C4, J1, J2, J5, J6, J7, J8, U1, U3, U4

Commit message: routing
Parts:
- added H1, H2, H3, H4: MountingHole, MountingHole:MountingHole_3.2mm_M3, symbol Mechanical:MountingHole
- renumbered J23 to J10, J22 to J8, J8 to J9, JP3 to JP2, JP2 to JP3, R34 to R1, R2 to R10, R3 to R11, R4 to R12, R5 to R13, R6 to R14, R7 to R15, R8 to R16, R9 to R17, R10 to R18, R11 to R19, R35 to R2, R12 to R20, R13 to R21, R14 to R22, R15 to R23, R16 to R24, R36 to R3, R37 to R4, R38 to R5, R39 to R6, R40 to R7, R41 to R8, R1 to R9
