File: UART-Multiplex.kicad_sch (KiCad schematic)
At the start: 7 parts, among them J14 Conn_01x08, J15 Conn_01x08, U3 74HC4051, U4 74HC4051

Commit message: updated schematics etc
Parts:
- removed J14, J15: Conn_01x08, symbol Connector_Generic:Conn_01x08
- added C10, C11, C12, C13, C14, C15, C9: 10uF, SparkFun-Capacitor:C_0603_1608Metric, symbol SparkFun-Capacitor:C
- added J13: TX/RX_CONN, Connector_PinHeader_1.00mm:PinHeader_1x03_P1.00mm_Vertical, symbol Connector_Generic:Conn_01x03
- added J14: NFC_CONN_0, Connector_JST:JST_XH_B4B-XH-A_1x04_P2.50mm_Vertical, symbol Connector_Generic:Conn_01x04
- added J15: NFC_CONN_1, Connector_JST:JST_XH_B4B-XH-A_1x04_P2.50mm_Vertical, symbol Connector_Generic:Conn_01x04
- added J16: NFC_CONN_2, Connector_JST:JST_XH_B4B-XH-A_1x04_P2.50mm_Vertical, symbol Connector_Generic:Conn_01x04
- added J17: NFC_CONN_3, Connector_JST:JST_XH_B4B-XH-A_1x04_P2.50mm_Vertical, symbol Connector_Generic:Conn_01x04
- added J18: NFC_CONN_4, Connector_JST:JST_XH_B4B-XH-A_1x04_P2.50mm_Vertical, symbol Connector_Generic:Conn_01x04
- added J19: NFC_CONN_5, Connector_JST:JST_XH_B4B-XH-A_1x04_P2.50mm_Vertical, symbol Connector_Generic:Conn_01x04
- added J24, J25: Conn_01x02, Connector_PinHeader_2.54mm:PinHeader_1x02_P2.54mm_Vertical, symbol Connector_Generic:Conn_01x02
- added NT1, NT2, NT3, NT4, NT5, NT6, NT7: NetTie_2, NetTie:NetTie-2_SMD_Pad0.5mm, symbol Device:NetTie_2
- added R18, R19, R20, R21, R22, R23, R24, R25, R26, R27, R28, R31: 4.7k, Resistor_SMD:R_0201_0603Metric_Pad0.64x0.40mm_HandSolder, symbol Device:R
- U7: renamed from U3; footprint Package_SO:SSOP-16_5.3x6.2mm_P0.65mm -> Package_SO:SOIC-16_3.9x9.9mm_P1.27mm
- U8: renamed from U4; footprint Package_SO:SSOP-16_5.3x6.2mm_P0.65mm -> Package_SO:SOIC-16_3.9x9.9mm_P1.27mm
- renumbered C2 to C6, C3 to C7, C6 to C8
Connections:
- net GND: now also C10.2, C11.2, C12.2, C13.2, C14.2, C15.2, C9.2, J13.1 (Pin_1), J14.1 (Pin_1), J15.1 (Pin_1), J16.1 (Pin_1), J17.1 (Pin_1), J18.1 (Pin_1), J19.1 (Pin_1), NT7.1, NT7.2
- net S0: now also NT1.2
- net S1: now also NT2.2
- net S2: now also NT3.2
- net NFC_TX_1: now reaches U7.13 (A0)
- net NFC_TX_1: now also J15.2 (Pin_2), R19.2
- net NFC_TX_2: now reaches U7.14 (A1)
- net NFC_TX_2: now also J16.2 (Pin_2), R20.2
- net NFC_TX_3: now reaches U7.15 (A2)
- net NFC_TX_3: now also J17.2 (Pin_2), R21.2
- net NFC_TX_0: now reaches U7.12 (A3)
- net NFC_TX_0: now also J14.2 (Pin_2), R18.2
- net NFC_TX_4: now reaches U7.1 (A4)
- net NFC_TX_4: now also J18.2 (Pin_2), R22.2
- net NFC_TX_7: now reaches U7.5 (A5)
- net NFC_TX_7: now also J25.1 (Pin_1)
- net NFC_TX_5: now reaches U7.2 (A6)
- net NFC_TX_5: now also J19.2 (Pin_2), R28.2
- net NFC_TX_6: now reaches U7.4 (A7)
- net NFC_TX_6: now also J24.1 (Pin_1)
- net NFC_RX_4: now reaches U8.1 (A4)
- net NFC_RX_4: now also J18.3 (Pin_3), R27.2
- net NFC_RX_0: now reaches U8.12 (A3)
- net NFC_RX_0: now also J14.3 (Pin_3), R23.2
- net NFC_RX_1: now reaches U8.13 (A0)
- net NFC_RX_1: now also J15.3 (Pin_3), R24.2
- net NFC_RX_2: now reaches U8.14 (A1)
- net NFC_RX_2: now also J16.3 (Pin_3), R25.2
- net NFC_RX_3: now reaches U8.15 (A2)
- net NFC_RX_3: now also J17.3 (Pin_3), R26.2
- net NFC_RX_5: now reaches U8.2 (A6)
- net NFC_RX_5: now also J19.3 (Pin_3), R31.2
- net NFC_RX_6: now reaches U8.4 (A7)
- net NFC_RX_6: now also J24.2 (Pin_2)
- net NFC_RX_7: now reaches U8.5 (A5)
- net NFC_RX_7: now also J25.2 (Pin_2)
- net 3.3v renamed 3.3V
- net 3.3V: now also C10.1, C11.1, C12.1, C13.1, C14.1, C15.1, C9.1, J14.4 (Pin_4), J15.4 (Pin_4), J16.4 (Pin_4), J17.4 (Pin_4), J18.4 (Pin_4), J19.4 (Pin_4), NT6.1, NT6.2, R18.1, R19.1, R20.1, R21.1, R22.1, R23.1, R24.1, R25.1, R26.1, R27.1, R28.1, R31.1
- net GPIO4 renamed MUX_TX
- net MUX_TX: now also J13.2 (Pin_2), NT4.2
- net GPIO6 renamed MUX_RX
- net MUX_RX: now also J13.3 (Pin_3), NT5.2
- new net GPIO11: NT4.1
- new net GPIO12: NT5.1
- new net GPIO13: NT1.1
- new net GPIO14: NT2.1
- new net GPIO15: NT3.1
Other:
- note added: "Decoupling Caps"
- note added: "Decoupling Caps for TXn/RXn Lines (Optional)"
- note added: "Pull-ups for TXn/RXn Lines (Optional)"
- moved on the sheet: C6, C7, C8, U7, U8

Commit message: routing
Parts:
- removed J13: TX/RX_CONN, Connector_PinHeader_1.00mm:PinHeader_1x03_P1.00mm_Vertical, symbol Connector_Generic:Conn_01x03
- removed J24, J25: Conn_01x02, Connector_PinHeader_2.54mm:PinHeader_1x02_P2.54mm_Vertical, symbol Connector_Generic:Conn_01x02
- removed NT1, NT2, NT3, NT4, NT5: NetTie_2, NetTie:NetTie-2_SMD_Pad0.5mm, symbol Device:NetTie_2
- added J14, J15, J16, J23, J24, J25, J26: Conn_01x01, Connector_PinHeader_2.54mm:PinHeader_1x01_P2.54mm_Vertical, symbol Connector_Generic:Conn_01x01
- renumbered C11 to C10, C12 to C11, C13 to C12, C14 to C13, C15 to C14, C6 to C5, C7 to C6, C8 to C7, C9 to C8, C10 to C9, J14 to J17, J15 to J18, J16 to J19, J17 to J20, J18 to J21, J19 to J22, NT6 to NT1, NT7 to NT2, R18 to R25, R19 to R26, R20 to R27, R21 to R28, R22 to R29, R23 to R30, R24 to R31, R25 to R32, R26 to R33, R27 to R34, R28 to R35, R31 to R36, U7 to U6, U8 to U7
Connections:
- net MUX_RX is gone; now on net GPIO12: U7.3 (A)
- net MUX_TX is gone; now on net GPIO11: U6.3 (A)
- net S0 is gone; now on net GPIO13: U6.11 (S0), U7.11 (S0)
- net S1 is gone; now on net GPIO14: U6.10 (S1), U7.10 (S1)
- net S2 is gone; now on net GPIO15: U6.9 (S2), U7.9 (S2)
- net GND: now also J14.1 (Pin_1)
- net GPIO11: now also J15.1 (Pin_1)
- net GPIO12: now also J16.1 (Pin_1)
- net NFC_RX_0: now also U7.13 (A0); no longer U7.12 (A3)
- net NFC_RX_1: now also U7.14 (A1); no longer U7.13 (A0)
- net NFC_RX_2: now also U7.15 (A2); no longer U7.14 (A1)
- net NFC_RX_3: now also U7.12 (A3); no longer U7.15 (A2)
- net NFC_RX_5: now also U7.5 (A5); no longer U7.2 (A6)
- net NFC_RX_6: now also U7.2 (A6), J24.1 (Pin_1); no longer U7.4 (A7)
- net NFC_RX_7: now also U7.4 (A7), J26.1 (Pin_1); no longer U7.5 (A5)
- net NFC_TX_0: now also U6.13 (A0); no longer U6.12 (A3)
- net NFC_TX_1: now also U6.14 (A1); no longer U6.13 (A0)
- net NFC_TX_2: now also U6.15 (A2); no longer U6.14 (A1)
- net NFC_TX_3: now also U6.12 (A3); no longer U6.15 (A2)
- net NFC_TX_5: now also U6.5 (A5); no longer U6.2 (A6)
- net NFC_TX_6: now also U6.2 (A6), J23.1 (Pin_1); no longer U6.4 (A7)
- net NFC_TX_7: now also U6.4 (A7), J25.1 (Pin_1); no longer U6.5 (A5)
