File: sp3485.kicad_sch (KiCad schematic)
At the start: 9 parts, among them J9 SP3485_PINS, U6 SP3485CN

Commit message: routing
Parts:
- renumbered C5 to C15, J9 to J27, JP6 to JP4, JP8 to JP5, JP7 to JP6, JP4 to JP7, JP5 to JP8, R17 to R37, U6 to U8
Changed lines of the file:
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@@
 		(dnp no)
 		(fields_autoplaced yes)
-		(property "Reference" "U6"
+		(property "Reference" "U8"
 			(at 83.4233 38.1 0)
 			(effects
@@
 			(project "ScrapheapPicoPCB"
 				(path "/0a0126d3-e10a-434c-bfa7-71e9aafa3ff9/95a9c5b6-9fe0-49f9-8813-a8150d9a6bbc/3cc70c3e-31db-4a59-99b0-9b2fed396c37"
-					(reference "U6")
+					(reference "U8")
 					(unit 1)
 				)
@@
 		(dnp no)
 		(fields_autoplaced yes)
-		(property "Reference" "#PWR027"
+		(property "Reference" "#PWR058"
 			(at 124.46 49.53 0)
 			(effects
@@
 			(project "ScrapheapPicoPCB"
 				(path "/0a0126d3-e10a-434c-bfa7-71e9aafa3ff9/95a9c5b6-9fe0-49f9-8813-a8150d9a6bbc/3cc70c3e-31db-4a59-99b0-9b2fed396c37"
-					(reference "#PWR027")
+					(reference "#PWR058")
 					(unit 1)
 				)
@@
 		(dnp no)
 		(fields_autoplaced yes)
-		(property "Reference" "#PWR024"
+		(property "Reference" "#PWR057"
 			(at 81.28 77.47 0)
 			(effects
@@
 			(project "ScrapheapPicoPCB"
 				(path "/0a0126d3-e10a-434c-bfa7-71e9aafa3ff9/95a9c5b6-9fe0-49f9-8813-a8150d9a6bbc/3cc70c3e-31db-4a59-99b0-9b2fed396c37"
-					(reference "#PWR024")
+					(reference "#PWR057")
 					(unit 1)
 				)
@@
 		(dnp no)
 		(fields_autoplaced yes)
-		(property "Reference" "JP4"
+		(property "Reference" "JP7"
 			(at 111.76 38.1 0)
 			(effects
@@
 			(project "ScrapheapPicoPCB"
 				(path "/0a0126d3-e10a-434c-bfa7-71e9aafa3ff9/95a9c5b6-9fe0-49f9-8813-a8150d9a6bbc/3cc70c3e-31db-4a59-99b0-9b2fed396c37"
-					(reference "JP4")
+					(reference "JP7")
 					(unit 1)
 				)
@@
 		(on_board yes)
 		(dnp no)
-		(property "Reference" "JP7"
+		(property "Reference" "JP6"
 			(at 60.96 67.31 0)
 			(effects
@@
 			(project "ScrapheapPicoPCB"
 				(path "/0a0126d3-e10a-434c-bfa7-71e9aafa3ff9/95a9c5b6-9fe0-49f9-8813-a8150d9a6bbc/3cc70c3e-31db-4a59-99b0-9b2fed396c37"
-					(reference "JP7")
+					(reference "JP6")
 					(unit 1)
 				)
@@
 		(on_board yes)
 		(dnp no)
-		(property "Reference" "#PWR028"
+		(property "Reference" "#PWR059"
 			(at 124.46 59.69 0)
 			(effects
@@
 			(project "ScrapheapPicoPCB"
 				(path "/0a0126d3-e10a-434c-bfa7-71e9aafa3ff9/95a9c5b6-9fe0-49f9-8813-a8150d9a6bbc/3cc70c3e-31db-4a59-99b0-9b2fed396c37"
-					(reference "#PWR028")
+					(reference "#PWR059")
 					(unit 1)
 				)
@@
 		(on_board yes)
 		(dnp no)
-		(property "Reference" "J9"
+		(property "Reference" "J27"
 			(at 36.83 38.1001 0)
 			(effects
@@
 			(project "ScrapheapPicoPCB"
 				(path "/0a0126d3-e10a-434c-bfa7-71e9aafa3ff9/95a9c5b6-9fe0-49f9-8813-a8150d9a6bbc/3cc70c3e-31db-4a59-99b0-9b2fed396c37"
-					(reference "J9")
+					(reference "J27")
 					(unit 1)
 				)
@@
 		(dnp no)
 		(fields_autoplaced yes)
-		(property "Reference" "JP5"
+		(property "Reference" "JP8"
 			(at 111.76 50.8 0)
 			(effects
@@
 			(project "ScrapheapPicoPCB"
 				(path "/0a0126d3-e10a-434c-bfa7-71e9aafa3ff9/95a9c5b6-9fe0-49f9-8813-a8150d9a6bbc/3cc70c3e-31db-4a59-99b0-9b2fed396c37"
-					(reference "JP5")
+					(reference "JP8")
 					(unit 1)
 				)
@@
 		(dnp no)
 		(fields_autoplaced yes)
-		(property "Reference" "JP6"
+		(property "Reference" "JP4"
 			(at 60.96 44.45 0)
 			(effects
@@
 			(project "ScrapheapPicoPCB"
 				(path "/0a0126d3-e10a-434c-bfa7-71e9aafa3ff9/95a9c5b6-9fe0-49f9-8813-a8150d9a6bbc/3cc70c3e-31db-4a59-99b0-9b2fed396c37"
-					(reference "JP6")
+					(reference "JP4")
 					(unit 1)
 				)
@@
 		(dnp no)
 		(fields_autoplaced yes)
-		(property "Reference" "#PWR021"
+		(property "Reference" "#PWR055"
 			(at 50.8 39.37 0)
 			(effects
@@
 			(project "ScrapheapPicoPCB"
 				(path "/0a0126d3-e10a-434c-bfa7-71e9aafa3ff9/95a9c5b6-9fe0-49f9-8813-a8150d9a6bbc/3cc70c3e-31db-4a59-99b0-9b2fed396c37"
-					(reference "#PWR021")
+					(reference "#PWR055")
 					(unit 1)
 				)
@@
 		(dnp no)
 		(fields_autoplaced yes)
-		(property "Reference" "C5"
+		(property "Reference" "C15"
 			(at 127 45.7262 0)
 			(effects
@@
 			(project "ScrapheapPicoPCB"
 				(path "/0a0126d3-e10a-434c-bfa7-71e9aafa3ff9/95a9c5b6-9fe0-49f9-8813-a8150d9a6bbc/3cc70c3e-31db-4a59-99b0-9b2fed396c37"
-					(reference "C5")
+					(reference "C15")
 					(unit 1)
 				)
@@
 		(dnp no)
 		(fields_autoplaced yes)
-		(property "Reference" "R17"
+		(property "Reference" "R37"
 			(at 106.68 49.5299 0)
 			(effects
@@
 			(project "ScrapheapPicoPCB"
 				(path "/0a0126d3-e10a-434c-bfa7-71e9aafa3ff9/95a9c5b6-9fe0-49f9-8813-a8150d9a6bbc/3cc70c3e-31db-4a59-99b0-9b2fed396c37"
-					(reference "R17")
+					(reference "R37")
 					(unit 1)
 				)
@@
 		(dnp no)
 		(fields_autoplaced yes)
-		(property "Reference" "JP8"
+		(property "Reference" "JP5"
 			(at 60.96 49.53 0)
 			(effects
@@
 			(project "ScrapheapPicoPCB"
 				(path "/0a0126d3-e10a-434c-bfa7-71e9aafa3ff9/95a9c5b6-9fe0-49f9-8813-a8150d9a6bbc/3cc70c3e-31db-4a59-99b0-9b2fed396c37"
-					(reference "JP8")
+					(reference "JP5")
 					(unit 1)
 				)
@@
 		(dnp no)
 		(fields_autoplaced yes)
-		(property "Reference" "#PWR023"
+		(property "Reference" "#PWR056"
 			(at 81.28 33.02 0)
 			(effects
@@
 			(project "ScrapheapPicoPCB"
 				(path "/0a0126d3-e10a-434c-bfa7-71e9aafa3ff9/95a9c5b6-9fe0-49f9-8813-a8150d9a6bbc/3cc70c3e-31db-4a59-99b0-9b2fed396c37"
-					(reference "#PWR023")
-					(unit 1)
-				)
+					(reference "#PWR056")
+					(unit 1)
+				)
